File: board/ESP32 Galvo Driver.kicad_sch (KiCad schematic)
At the start: 75 parts, among them J1 15V Power In, J10 15V Supply In, J11 AudioJack3_SwitchTR, J12 LASER_EN, J13 FAN, J2 RED, J3 GREEN, J4 BLUE, J5 Native USB, J6 Galvo X Output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

Commit message: ILDA test pattern WIP
Connections:
- net GND: no longer U1.1 (GND), U1.40 (GND), U1.41 (GND)
- new net: U1.1 (GND), U1.40 (GND), U1.41 (GND)
Other:
- note added: "+/-15V Power Input"
- note added: "12V -> 3.3V Regulation"
- note added: "AC 120V/240V Power Input"
- note added: "Enclosure"
- note added: "Galvo Signal Handling"
- note added: "Laser Control"
- note added: "Microcontroller and Debug"
- note added: "Power Regulation"
- note added: "Wii Accessory Connectors"
- note removed: "3.3V Regulation"
- note removed: "Nunchucks"
- note removed: "Power Input"
- moved on the sheet: C1, C2, C3, C4, C5, C6, C7, C8, C9, D1, D2, D3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

Commit message: update board
Parts:
- added J14: Laser Key, Connector_JST:JST_XH_B2B-XH-A_1x02_P2.50mm_Vertical, symbol Connector_Generic:Conn_01x02
- added J15: Conn_01x05, Connector_PinHeader_2.54mm:PinHeader_1x05_P2.54mm_Vertical, symbol Connector_Generic:Conn_01x05
- added J16: Quiic 1, Connector_JST:JST_SH_BM04B-SRSS-TB_1x04-1MP_P1.00mm_Vertical, symbol Connector_Generic_MountingPin:Conn_01x04_MountingPin
- added J17: Quiic 2, Connector_JST:JST_SH_BM04B-SRSS-TB_1x04-1MP_P1.00mm_Vertical, symbol Connector_Generic_MountingPin:Conn_01x04_MountingPin
- added JP1: DAC X Select, Jumper:SolderJumper-3_P1.3mm_Bridged12_RoundedPad1.0x1.5mm, symbol Jumper:SolderJumper_3_Bridged12
- added JP2: DAC Y Select, Jumper:SolderJumper-3_P1.3mm_Bridged12_RoundedPad1.0x1.5mm, symbol Jumper:SolderJumper_3_Bridged12
- added JP3: Key Bypass, Jumper:SolderJumper-2_P1.3mm_Open_TrianglePad1.0x1.5mm, symbol Jumper:SolderJumper_2_Open
- added R30: 100k, Resistor_SMD:R_0603_1608Metric_Pad0.98x0.95mm_HandSolder, symbol Device:R
- added R31: 27k, Resistor_SMD:R_0603_1608Metric_Pad0.98x0.95mm_HandSolder, symbol Device:R
- added U5: MCP4922-ESL, Package_SO:SOIC-14_3.9x8.7mm_P1.27mm, symbol Analog_DAC:MCP4922-ESL
- P1: value CONN_WII -> Wii 1
- P2: value CONN_WII -> Wii 2
Connections:
- net +12V: now also J14.2 (Pin_2), JP3.1 (A); no longer Q3.2 (S), R24.2
- net +3.3V: now also J16.2 (Pin_2), J17.2 (Pin_2), U5.1 (VDD), U5.11 (VrefB), U5.13 (VrefA), U5.9 (~{SHDN})
- net DAC_X: now also JP1.2 (C); no longer U1.10 (GPIO17/U1TXD/ADC2_CH6/DAC_1)
- net DAC_Y: now also JP2.2 (C); no longer U1.11 (GPIO18/U1RXD/ADC2_CH7/DAC_2/CLK_OUT3)
- net DTR: now also J15.2 (Pin_2)
- net GND: now also U1.1 (GND), U1.40 (GND), U1.41 (GND), J15.1 (Pin_1), J16.1 (Pin_1), J16.MP (MountPin), J17.1 (Pin_1), J17.MP (MountPin), R31.2, U5.12 (AVSS), U5.8 (~{LDAC})
- net I2C0_SCL: now also J16.4 (Pin_4)
- net I2C0_SDA: now also J16.3 (Pin_3)
- net I2C1_SCL: now also J17.4 (Pin_4)
- net I2C1_SDA: now also J17.3 (Pin_3)
- net RTS: now also J15.3 (Pin_3)
- net UART_RX: now also J15.4 (Pin_4)
- net UART_TX: now also J15.5 (Pin_5)
- net KEY_SENSE: now reaches U1.17 (GPIO9/TOUCH9/ADC1_CH8/FSPIHD)
- net KEY_SENSE: now also R30.2, R31.1
- net SPI_CS_DAC: now reaches U1.25 (SPIIO5/GPIO34/FSPICS0)
- net SPI_CS_DAC: now also U5.3 (~{CS})
- net SPI_MOSI: now reaches U1.28 (SPIIO6/GPIO35/FSPID)
- net SPI_MOSI: now also U5.5 (SDI)
- net SPI_SCK: now reaches U1.29 (SPIIO7/GPIO36/FSPICLK)
- net SPI_SCK: now also U5.4 (SCK)
- net SPI_MISO: now reaches U1.30 (SPIDQS/GPIO37/FSPIQ)
- new net: J14.1 (Pin_1), JP3.2 (B), Q3.2 (S), R24.2, R30.1
- new net DAC_X_EXT: JP1.3 (B), U5.14 (VoutA)
- new net DAC_X_INT: JP1.1 (A), U1.10 (GPIO17/U1TXD/ADC2_CH6/DAC_1)
- new net DAC_Y_EXT: JP2.3 (B), U5.10 (VoutB)
- new net DAC_Y_INT: JP2.1 (A), U1.11 (GPIO18/U1RXD/ADC2_CH7/DAC_2/CLK_OUT3)
Other:
- note added: "I2C and Wii Accessory Connectors"
- note added: "UART Header"
- note removed: "Wii Accessory Connectors"
- moved on the sheet: C8, C9, J11, J12, P1, P2, Q3, Q4, R24, R25, U1

Commit message: gtfs, litt.chr parsing
Parts:
- added C10: 10uF, Capacitor_SMD:C_0603_1608Metric_Pad1.08x0.95mm_HandSolder, symbol Device:C
- added C11: 0.1uF, Capacitor_SMD:C_0603_1608Metric_Pad1.08x0.95mm_HandSolder, symbol Device:C
Connections:
- net +3.3V: now also C10.1, C11.1
- net GND: now also C10.2, C11.2

Commit message: switch to pinouts from PCB, separate package for vector text
Parts:
- added JP4: UART_RX, Jumper:SolderJumper-2_P1.3mm_Bridged_Pad1.0x1.5mm, symbol Jumper:SolderJumper_2_Bridged
- added JP5: UART_TX, Jumper:SolderJumper-2_P1.3mm_Bridged_Pad1.0x1.5mm, symbol Jumper:SolderJumper_2_Bridged
- added R32, R33, R34, R35: 10k, Resistor_SMD:R_0603_1608Metric_Pad0.98x0.95mm_HandSolder, symbol Device:R
- added TP1: 12V, TestPoint:TestPoint_Pad_D2.5mm, symbol Connector:TestPoint
- added TP2: 3.3V, TestPoint:TestPoint_Pad_D2.5mm, symbol Connector:TestPoint
Connections:
- net +12V: now also TP1.1
- net +3.3V: now also R32.1, R33.1, R34.1, R35.1, TP2.1
- net I2C0_SCL: now also R32.2
- net I2C0_SDA: now also R33.2
- net I2C1_SCL: now also R34.2
- net I2C1_SDA: now also R35.2
- net UART_RX: now also JP4.2 (B); no longer U2.26 (TXD)
- net UART_TX: now also JP5.2 (B); no longer U2.25 (RXD)
- new net: JP4.1 (A), U2.26 (TXD)
- new net: JP5.1 (A), U2.25 (RXD)

Commit message: board updates: fix improper wiring of AC input
Parts:
- U4: value ~ -> (none)
